Commit message: Gazebo sim init

File: description/robot.urdf.xacro (robot description, xacro)
@@ -3,3 +3,4 @@
     <xacro:include filename="inertial_macros.xacro" />
     <xacro:include filename="robot_core.xacro" />
+    <xacro:include filename="gazebo_control.xacro" />
 </robot>

File: description/robot_core.xacro (robot description, xacro)
@@ -20,5 +20,5 @@
         <parent link="base_link"/>
         <child link="chassis"/>
-        <origin xyz="0 0 0.020"/>
+        <origin xyz="0 0 0.037"/>
     </joint>
     <link name="chassis">
@@ -37,7 +37,10 @@
         </collision>
         <xacro:inertial_cylinder mass="1.23" length="0.11" radius="0.09">
-            <origin xyz="0.15 0 0.075" rpy="0 0 0"/>
+            <origin xyz="0 0 0.035" rpy="0 0 0"/>
         </xacro:inertial_cylinder>
     </link>
+    <gazebo reference="chassis">
+        <material>Gazebo/White</material>
+    </gazebo>
     <!-- LEFT WHEEL -->
     <joint name="left_wheel_joint" type="continuous">
@@ -48,5 +51,5 @@
     </joint>
     <link name="left_wheel">
-        <visual>
+        <!--visual>
             <origin xyz="0 0 0.0065" rpy="0 0 0"/>
             <geometry>
@@ -54,9 +57,9 @@
             </geometry>
             <material name="blue"/>
-        </visual>
+        </visual-->
         <visual>
-            <origin xyz="0 0 0.0285" rpy="0 0 0"/>
+            <origin xyz="0 0 0.022" rpy="0 0 0"/>
             <geometry>
-                <cylinder length="0.031" radius="0.037" />
+                <cylinder length="0.044" radius="0.037" />
             </geometry>
             <material name="blue"/>
@@ -73,4 +76,7 @@
         </xacro:inertial_cylinder>
     </link>
+    <gazebo reference="left_wheel">
+        <material>Gazebo/Blue</material>
+    </gazebo>
     <!-- RIGHT WHEEL -->
     <joint name="right_wheel_joint" type="continuous">
@@ -81,5 +87,5 @@
     </joint>
     <link name="right_wheel">
-        <visual>
+        <!--visual>
             <origin xyz="0 0 0.0065" rpy="0 0 0"/>
             <geometry>
@@ -87,9 +93,9 @@
             </geometry>
             <material name="blue"/>
-        </visual>
+        </visual-->
         <visual>
-            <origin xyz="0 0 0.0285" rpy="0 0 0"/>
+            <origin xyz="0 0 0.022" rpy="0 0 0"/>
             <geometry>
-                <cylinder length="0.031" radius="0.037" />
+                <cylinder length="0.044" radius="0.037" />
             </geometry>
             <material name="blue"/>
@@ -106,9 +112,12 @@
         </xacro:inertial_cylinder>
     </link>
+    <gazebo reference="right_wheel">
+        <material>Gazebo/Blue</material>
+    </gazebo>
     <!-- FRONT CASTER WHEEL -->
     <joint name="front_caster_wheel_joint" type="fixed">
         <parent link="base_link"/>
         <child link="front_caster_wheel"/>
-        <origin xyz="0.076 0 0" rpy="0 0 0"/>
+        <origin xyz="0.076 0 0.017" rpy="0 0 0"/>
     </joint>
     <link name="front_caster_wheel">
@@ -129,9 +138,14 @@
         </xacro:inertial_sphere>
     </link>
+    <gazebo reference="front_caster_wheel">
+        <material>Gazebo/Black</material>
+        <mu1 value="0.001"/>
+        <mu2 value="0.001"/>
+    </gazebo>
     <!-- BACK CASTER WHEEL -->
     <joint name="back_caster_wheel_joint" type="fixed">
         <parent link="base_link"/>
         <child link="back_caster_wheel"/>
-        <origin xyz="-0.076 0 0" rpy="0 0 0"/>
+        <origin xyz="-0.076 0 0.017" rpy="0 0 0"/>
     </joint>
     <link name="back_caster_wheel">
@@ -152,3 +166,8 @@
         </xacro:inertial_sphere>
     </link>
+    <gazebo reference="back_caster_wheel">
+        <material>Gazebo/Blue</material>
+        <mu1 value="0.001"/>
+        <mu2 value="0.001"/>
+    </gazebo>
 </robot>
