Commit message: odometry fixes

File: description/robot_core.xacro (robot description, xacro)
@@ -59,19 +59,19 @@
         </visual-->
         <visual>
-            <origin xyz="0 0 0.022" rpy="0 0 0"/>
+            <origin xyz="0 0 0.0165" rpy="0 0 0"/>
             <geometry>
-                <cylinder length="0.044" radius="0.037" />
+                <cylinder length="0.031" radius="0.037" />
             </geometry>
             <material name="blue"/>
         </visual>
         <collision>
-            <origin xyz="0 0 0.022" rpy="0 0 0"/>
+            <origin xyz="0 0 0.0165" rpy="0 0 0"/>
             <geometry>
-                <cylinder length="0.044" radius="0.037" />
+                <cylinder length="0.031" radius="0.037" />
             </geometry>
             <material name="blue"/>
         </collision>
-        <xacro:inertial_cylinder mass="0.035" length="0.044" radius="0.037">
-            <origin xyz="0 0 0.022" rpy="0 0 0"/>
+        <xacro:inertial_cylinder mass="0.035" length="0.031" radius="0.037">
+            <origin xyz="0 0 0.0165" rpy="0 0 0"/>
         </xacro:inertial_cylinder>
     </link>
@@ -95,19 +95,19 @@
         </visual-->
         <visual>
-            <origin xyz="0 0 0.022" rpy="0 0 0"/>
+            <origin xyz="0 0 0.0165" rpy="0 0 0"/>
             <geometry>
-                <cylinder length="0.044" radius="0.037" />
+                <cylinder length="0.031" radius="0.037" />
             </geometry>
             <material name="blue"/>
         </visual>
         <collision>
-            <origin xyz="0 0 0.022" rpy="0 0 0"/>
+            <origin xyz="0 0 0.0165" rpy="0 0 0"/>
             <geometry>
-                <cylinder length="0.044" radius="0.037" />
+                <cylinder length="0.031" radius="0.037" />
             </geometry>
             <material name="blue"/>
         </collision>
-        <xacro:inertial_cylinder mass="0.035" length="0.044" radius="0.037">
-            <origin xyz="0 0 0.022" rpy="0 0 0"/>
+        <xacro:inertial_cylinder mass="0.035" length="0.031" radius="0.037">
+            <origin xyz="0 0 0.0165" rpy="0 0 0"/>
         </xacro:inertial_cylinder>
     </link>

File: description/ros2_control.xacro (robot description, xacro)
@@ -11,10 +11,10 @@
                 <param name="baud_rate">57600</param>
                 <param name="timeout">1000</param>
-                <param name="enc_counts_per_rev">2150</param>
+                <param name="enc_counts_per_rev">2154</param>
             </hardware>
             <joint name="left_wheel_joint">
                 <command_interface name="velocity">
-                    <param name="min">-10</param>
-                    <param name="max">10</param>
+                    <param name="min">-18</param>
+                    <param name="max">18</param>
                 </command_interface>
                 <state_interface name="position" />
@@ -23,6 +23,6 @@
             <joint name="right_wheel_joint">
                 <command_interface name="velocity">
-                    <param name="min">-10</param>
-                    <param name="max">10</param>
+                    <param name="min">-15</param>
+                    <param name="max">15</param>
                 </command_interface>
                 <state_interface name="velocity" />
